Commit message: rosserial

File: caddy_bot/urdf/tf_follow_caddy_bot.urdf.xacro (robot description, xacro)
@@ -41,3 +41,9 @@
   </joint>
   <link name="camera_link"/>
+  <joint name="uwb_joint" type="fixed">
+    <parent link="base_link"/>
+    <child link="uwb_link"/>
+    <origin xyz="0.0 0.0 0.0" rpy="0 0 0"/>
+  </joint>
+  <link name="uwb_link"/>
 </robot>
